File: pcb/skyear.kicad_sch (KiCad schematic)
At the start: 52 parts, among them J1 BATTERY, J2 ANTENNA, J3 PHONES, J4 LINE_OUT, SW1 POWER, U1 TL072, U2 TL072, U3 LM386N-1

Commit message: Use real DigiKey parts in BOM; switch SW1 to right-angle footprint
- bom.csv: every line now has the DigiKey part number and price from the
  actual cart (34 lines, $29.67 parts subtotal). Obsolete Nichicon caps and
  backordered parts were replaced with in-stock equivalents in the same sizes.
- SW1: the switch in the cart is the right-angle C&K OS102011MA1QN1, so the
  footprint is now SW_Slide_SPDT_Angled_CK_OS102011MA1Q (same pins 1/2/3).
  ERC: 0 errors; netlist and footprint pads re-verified.

Co-Authored-By: Claude Opus 5.5 <noreply@anthropic.com>
Claude-Session: https://claude.ai/code/session_017gCygh5QrYo9QD1FT88DS2
Parts:
- SW1: footprint Button_Switch_THT:SW_Slide_SPDT_Straight_CK_OS102011MS2Q -> Button_Switch_THT:SW_Slide_SPDT_Angled_CK_OS102011MA1Q; MPN C&K OS102011MS2QN1 -> C&K OS102011MA1QN1 (right-angle)
Changed lines of the file:
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@@
 			)
 		)
-		(property "Footprint" "Button_Switch_THT:SW_Slide_SPDT_Straight_CK_OS102011MS2Q"
+		(property "Footprint" "Button_Switch_THT:SW_Slide_SPDT_Angled_CK_OS102011MA1Q"
 			(at 60.96 40.64 0)
 			(effects
@@
 			)
 		)
-		(property "MPN" "C&K OS102011MS2QN1"
+		(property "MPN" "C&K OS102011MA1QN1 (right-angle)"
 			(at 60.96 40.64 0)
 			(effects
